Commit message: -

File: urdf/4_cameras_v1/4_cameras_v1.urdf.xacro (robot description, xacro)
@@ -9,6 +9,6 @@
     <xacro:property name="y_d" value="0.1"/>
     <!-- Base link-->
-<!--    <link name="sim_world"></link>-->
     <link name="base_link">
+        <kinematic>1</kinematic>
         <!-- pose and inertial -->
         <pose>0 0 0 0 0 0</pose>
@@ -32,4 +32,7 @@
         </visual>
     </link>
+    <gazebo reference="base_link">
+        <kinematic>1</kinematic>
+    </gazebo>
     <!-- Cameras  -->
     <xacro:macro name="hlp_camera" params="name xyz rpy">
@@ -42,4 +45,69 @@
         </joint>
     </xacro:macro>
+<!--    <link name="camera1_link">-->
+<!--        <collision>-->
+<!--            <origin xyz="0 0 0" rpy="0 0 0" />-->
+<!--            <geometry>-->
+<!--                <box size="0.04 0.04 0.04" />-->
+<!--            </geometry>-->
+<!--        </collision>-->
+<!--        <visual>-->
+<!--            <origin xyz="0 0 0" rpy="0 0 0" />-->
+<!--            <geometry>-->
+<!--                <box size="0.04 0.04 0.04" />-->
+<!--            </geometry>-->
+<!--            <material name="gray" />-->
+<!--        </visual>-->
+<!--        <inertial>-->
+<!--            <mass value="1e-5" />-->
+<!--            <origin xyz="0 0 0" rpy="0 0 0" />-->
+<!--            <inertia ixx="1e-6" ixy="0" ixz="0" iyy="1e-6" iyz="0" izz="1e-6" />-->
+<!--        </inertial>-->
+<!--    </link>-->
+<!--    <gazebo reference="camera1_link">-->
+<!--        <sensor type="camera" name="camera1">-->
+<!--            <update_rate>30.0</update_rate>-->
+<!--            <camera name="head">-->
+<!--                <horizontal_fov>1.2262634</horizontal_fov>-->
+<!--                <image>-->
+<!--                    <width>640</width>-->
+<!--                    <height>480</height>-->
+<!--                    <format>R8G8B8</format>-->
+<!--                </image>-->
+<!--                <clip>-->
+<!--                    <near>0.02</near>-->
+<!--                    <far>300</far>-->
+<!--                </clip>-->
+<!--                <noise>-->
+<!--                    <type>gaussian</type>-->
+<!--                    &lt;!&ndash; Noise is sampled independently per pixel on each frame.-->
+<!--               That pixel's noise value is added to each of its color-->
+<!--               channels, which at that point lie in the range [0,1]. &ndash;&gt;-->
+<!--                    <mean>0.0</mean>-->
+<!--                    <stddev>0.007</stddev>-->
+<!--                </noise>-->
+<!--            </camera>-->
+<!--            <plugin name="camera_controller" filename="libgazebo_ros_camera.so">-->
+<!--                <alwaysOn>true</alwaysOn>-->
+<!--                <updateRate>0.0</updateRate>-->
+<!--                <cameraName>camera1</cameraName>-->
+<!--                <imageTopicName>image_raw</imageTopicName>-->
+<!--                <cameraInfoTopicName>camera_info</cameraInfoTopicName>-->
+<!--                <frameName>/camera1_link</frameName>-->
+<!--                <hackBaseline>0.07</hackBaseline>-->
+<!--                <distortionK1>0.0</distortionK1>-->
+<!--                <distortionK2>0.0</distortionK2>-->
+<!--                <distortionK3>0.0</distortionK3>-->
+<!--                <distortionT1>0.0</distortionT1>-->
+<!--                <distortionT2>0.0</distortionT2>-->
+<!--            </plugin>-->
+<!--        </sensor>-->
+<!--    </gazebo>-->
+<!--    <joint name="camera_joint" type="fixed">-->
+<!--        <axis xyz="0 1 0" />-->
+<!--        <origin xyz="0.1 0.0 0.2" rpy="0 0.5 0" />-->
+<!--        <parent link="base_link" />-->
+<!--        <child link="camera1_link" />-->
+<!--    </joint>-->
     <xacro:hlp_camera name="camera_0" xyz="${x_d/2} ${y_d/2} 0" rpy="0 0 0" />
     <xacro:hlp_camera name="camera_1" xyz="${x_d/2} ${-y_d/2} 0" rpy="0 0 0" />

File: urdf/camera.urdf.xacro (robot description, xacro)
@@ -24,5 +24,5 @@
         </link>
         <gazebo reference="${name}_link">
-            <sensor type="camera" name="s_${name}">
+            <sensor type="camera" name="${name}">
                 <update_rate>${update_rate}</update_rate>
                 <camera name="${name}">
@@ -46,11 +46,10 @@
                     </noise>
                 </camera>
-                <plugin name="${name}_camera_controller" filename="libgazebo_ros_camera.so">
+                <plugin name="camera_controller" filename="libgazebo_ros_camera.so">
                     <alwaysOn>true</alwaysOn>
-                    <updateRate>${update_rate}</updateRate>
                     <cameraName>${name}</cameraName>
                     <imageTopicName>image_raw</imageTopicName>
                     <cameraInfoTopicName>camera_info</cameraInfoTopicName>
-                    <frameName>{name}_link</frameName>
+                    <frameName>${name}_link</frameName>
                     <hackBaseline>0.07</hackBaseline>
                     <distortionK1>0.0</distortionK1>

File: urdf/imu.urdf.xacro (robot description, xacro)
@@ -26,11 +26,10 @@
             <sensor name="s_${name}" type="imu">
                 <always_on>true</always_on>
-                <update_rate>${update_rate}</update_rate>
+                <update_rate>0.0</update_rate>
                 <visualize>true</visualize>
-                <topic>__default_topic__</topic>
                 <plugin filename="libgazebo_ros_imu_sensor.so" name="imu_plugin">
                     <topicName>${name}</topicName>
                     <bodyName>${name}_link</bodyName>
-                    <updateRateHZ>update_rate</updateRateHZ>
+                    <updateRateHZ>0.0</updateRateHZ>
                     <gaussianNoise>0.0</gaussianNoise>
                     <xyzOffset>0 0 0</xyzOffset>

Commit message: it is usable :)

File: urdf/4_cameras_v1/4_cameras_v1.urdf.xacro (robot description, xacro)
@@ -4,8 +4,8 @@
     <xacro:include filename="$(find v-nav-gazebo-sim)/urdf/camera.urdf.xacro" />
     <xacro:include filename="$(find v-nav-gazebo-sim)/urdf/imu.urdf.xacro" />
-    <xacro:property name="update_rate" value="30"/>
-    <xacro:property name="fov" value="1.22"/>
-    <xacro:property name="x_d" value="0.1"/>
-    <xacro:property name="y_d" value="0.1"/>
+<!--    <xacro:property name="update_rate" value="30"/>-->
+<!--    <xacro:property name="fov" value="${120 * pi / 180}"/>-->
+    <xacro:property name="x_d" value="0.12"/>
+    <xacro:property name="y_d" value="0.12"/>
     <!-- Base link-->
     <link name="base_link">
@@ -36,6 +36,7 @@
     </gazebo>
     <!-- Cameras  -->
-    <xacro:macro name="hlp_camera" params="name xyz rpy">
-        <xacro:camera name="${name}" update_rate="${update_rate}" fov="${fov}" />
+    <xacro:macro name="hlp_camera" params="name xyz rpy mat">
+<!--        <xacro:simple_camera name="${name}" />-->
+        <xacro:dist_camera name="${name}" />
         <joint name="${name}_joint" type="fixed">
             <axis xyz="0 1 0" />
@@ -44,74 +45,12 @@
             <child link="${name}_link"/>
         </joint>
+        <gazebo reference="${name}_link">
+            <material>${mat}</material>
+        </gazebo>
     </xacro:macro>
-<!--    <link name="camera1_link">-->
-<!--        <collision>-->
-<!--            <origin xyz="0 0 0" rpy="0 0 0" />-->
-<!--            <geometry>-->
-<!--                <box size="0.04 0.04 0.04" />-->
-<!--            </geometry>-->
-<!--        </collision>-->
-<!--        <visual>-->
-<!--            <origin xyz="0 0 0" rpy="0 0 0" />-->
-<!--            <geometry>-->
-<!--                <box size="0.04 0.04 0.04" />-->
-<!--            </geometry>-->
-<!--            <material name="gray" />-->
-<!--        </visual>-->
-<!--        <inertial>-->
-<!--            <mass value="1e-5" />-->
-<!--            <origin xyz="0 0 0" rpy="0 0 0" />-->
-<!--            <inertia ixx="1e-6" ixy="0" ixz="0" iyy="1e-6" iyz="0" izz="1e-6" />-->
-<!--        </inertial>-->
-<!--    </link>-->
-<!--    <gazebo reference="camera1_link">-->
-<!--        <sensor type="camera" name="camera1">-->
-<!--            <update_rate>30.0</update_rate>-->
-<!--            <camera name="head">-->
-<!--                <horizontal_fov>1.2262634</horizontal_fov>-->
-<!--                <image>-->
-<!--                    <width>640</width>-->
-<!--                    <height>480</height>-->
-<!--                    <format>R8G8B8</format>-->
-<!--                </image>-->
-<!--                <clip>-->
-<!--                    <near>0.02</near>-->
-<!--                    <far>300</far>-->
-<!--                </clip>-->
-<!--                <noise>-->
-<!--                    <type>gaussian</type>-->
-<!--                    &lt;!&ndash; Noise is sampled independently per pixel on each frame.-->
-<!--               That pixel's noise value is added to each of its color-->
-<!--               channels, which at that point lie in the range [0,1]. &ndash;&gt;-->
-<!--                    <mean>0.0</mean>-->
-<!--                    <stddev>0.007</stddev>-->
-<!--                </noise>-->
-<!--            </camera>-->
-<!--            <plugin name="camera_controller" filename="libgazebo_ros_camera.so">-->
-<!--                <alwaysOn>true</alwaysOn>-->
-<!--                <updateRate>0.0</updateRate>-->
-<!--                <cameraName>camera1</cameraName>-->
-<!--                <imageTopicName>image_raw</imageTopicName>-->
-<!--                <cameraInfoTopicName>camera_info</cameraInfoTopicName>-->
-<!--                <frameName>/camera1_link</frameName>-->
-<!--                <hackBaseline>0.07</hackBaseline>-->
-<!--                <distortionK1>0.0</distortionK1>-->
-<!--                <distortionK2>0.0</distortionK2>-->
-<!--                <distortionK3>0.0</distortionK3>-->
-<!--                <distortionT1>0.0</distortionT1>-->
-<!--                <distortionT2>0.0</distortionT2>-->
-<!--            </plugin>-->
-<!--        </sensor>-->
-<!--    </gazebo>-->
-<!--    <joint name="camera_joint" type="fixed">-->
-<!--        <axis xyz="0 1 0" />-->
-<!--        <origin xyz="0.1 0.0 0.2" rpy="0 0.5 0" />-->
-<!--        <parent link="base_link" />-->
-<!--        <child link="camera1_link" />-->
-<!--    </joint>-->
-    <xacro:hlp_camera name="camera_0" xyz="${x_d/2} ${y_d/2} 0" rpy="0 0 0" />
-    <xacro:hlp_camera name="camera_1" xyz="${x_d/2} ${-y_d/2} 0" rpy="0 0 0" />
-    <xacro:hlp_camera name="camera_2" xyz="${-x_d/2} ${-y_d/2} 0" rpy="0 0 0" />
-    <xacro:hlp_camera name="camera_3" xyz="${-x_d/2} ${y_d/2} 0" rpy="0 0 0" />
+    <xacro:hlp_camera name="camera_0" xyz="${x_d/2} ${y_d/2} 0" rpy="0 ${0} ${0}" mat="Gazebo/Yellow" />
+    <xacro:hlp_camera name="camera_1" xyz="${x_d/2} ${-y_d/2} 0" rpy="0 ${0} ${0}" mat="Gazebo/Orange"  />
+    <xacro:hlp_camera name="camera_2" xyz="${-x_d/2} ${y_d/2} 0" rpy="0 ${pi/10} ${pi-pi/2}" mat="Gazebo/Red"  />
+    <xacro:hlp_camera name="camera_3" xyz="${-x_d/2} ${-y_d/2} 0" rpy="0 ${pi/10} ${-pi+pi/2}" mat="Gazebo/Purple"  />
     <!-- IMU -->
     <xacro:imu name="imu" update_rate="100"/>

File: urdf/camera.urdf.xacro (robot description, xacro)
@@ -1,5 +1,5 @@
 <?xml version="1.0"?>
 <robot xmlns:xacro="http://www.ros.org/wiki/xacro">
-    <xacro:macro name="camera" params="name update_rate fov">
+    <xacro:macro name="camera_sensor_base" params="name width height update_rate horizontal_fov frame_name k1 k2 k3 p1 p2 cx cy cx_prime">
         <!-- Camera -->
         <link name="${name}_link">
@@ -7,5 +7,5 @@
                 <origin xyz="0 0 0" rpy="0 0 0"/>
                 <geometry>
-                    <box size="0.04 0.04 0.04"/>
+                    <box size="0.03 0.03 0.03"/>
                 </geometry>
             </collision>
@@ -13,5 +13,5 @@
                 <origin xyz="0 0 0" rpy="0 0 0"/>
                 <geometry>
-                    <box size="0.04 0.04 0.04"/>
+                    <box size="0.03 0.03 0.03"/>
                 </geometry>
                 <material name="red"/>
@@ -25,14 +25,15 @@
         <gazebo reference="${name}_link">
             <sensor type="camera" name="${name}">
+                <visualize>true</visualize>
                 <update_rate>${update_rate}</update_rate>
                 <camera name="${name}">
-                    <horizontal_fov>${fov}</horizontal_fov>
+                    <horizontal_fov>${horizontal_fov}</horizontal_fov>
                     <image>
-                        <width>640</width>
-                        <height>480</height>
+                        <width>${width}</width>
+                        <height>${height}</height>
                         <format>R8G8B8</format>
                     </image>
                     <clip>
-                        <near>0.02</near>
+                        <near>0.01</near>
                         <far>300</far>
                     </clip>
@@ -45,4 +46,12 @@
                         <stddev>0.007</stddev>
                     </noise>
+                    <distortion>
+                        <k1>${k1}</k1>
+                        <k2>${k2}</k2>
+                        <k3>${k3}</k3>
+                        <p1>${p1}</p1>
+                        <p2>${p2}</p2>
+                        <center>${(cx - 0.5)/ width} ${(cy - 0.5) / height}</center>
+                    </distortion>
                 </camera>
                 <plugin name="camera_controller" filename="libgazebo_ros_camera.so">
@@ -51,14 +60,60 @@
                     <imageTopicName>image_raw</imageTopicName>
                     <cameraInfoTopicName>camera_info</cameraInfoTopicName>
-                    <frameName>${name}_link</frameName>
-                    <hackBaseline>0.07</hackBaseline>
-                    <distortionK1>0.0</distortionK1>
-                    <distortionK2>0.0</distortionK2>
-                    <distortionK3>0.0</distortionK3>
-                    <distortionT1>0.0</distortionT1>
-                    <distortionT2>0.0</distortionT2>
+                    <frameName>${frame_name}</frameName>
+<!--                    <hackBaseline>0.07</hackBaseline>-->
+<!--                    <distortionK1>0.0</distortionK1>-->
+<!--                    <distortionK2>0.0</distortionK2>-->
+<!--                    <distortionK3>0.0</distortionK3>-->
+<!--                    <distortionT1>0.0</distortionT1>-->
+<!--                    <distortionT2>0.0</distortionT2>-->
+                    <CxPrime>${cx_prime}</CxPrime>
+                    <Cx>${cx}</Cx>
+                    <Cy>${cy}</Cy>
+                    <distortionK1>${k1}</distortionK1>
+                    <distortionK2>${k2}</distortionK2>
+                    <distortionK3>${k3}</distortionK3>
+                    <distortionT1>${p1}</distortionT1>
+                    <distortionT2>${p2}</distortionT2>
                 </plugin>
             </sensor>
         </gazebo>
     </xacro:macro>
+    <xacro:macro name="camera_sensor" params="name width height update_rate horizontal_fov k1:=0 k2:=0 k3:=0 p1:=0 p2:=0">
+        <xacro:camera_sensor_base
+                name="${name}"
+                width="${width}"
+                height="${height}"
+                update_rate="${update_rate}"
+                horizontal_fov="${horizontal_fov}"
+                frame_name="${name}_optical"
+                k1="${k1}"
+                k2="${k2}"
+                k3="${k3}"
+                p1="${p1}"
+                p2="${p2}"
+                cx="${(width + 1.0)/2.0}"
+                cy="${(height + 1.0)/2.0}"
+                cx_prime="${(width + 1.0)/2.0}"
+        />
+    </xacro:macro>
+    <xacro:macro name="simple_camera" params="name">
+        <xacro:camera_sensor name="${name}" width="640" height="480" update_rate="30" horizontal_fov="${120.0*pi/180.0}"/>
+    </xacro:macro>
+    <xacro:macro name="dist_camera" params="name">
+        <xacro:camera_sensor_base name="${name}"
+                                  frame_name="/${name}_optical"
+                                  width="320"
+                                  height="240"
+                                  update_rate="30"
+                                  horizontal_fov="1.8"
+                                  k1="-0.273377"
+                                  k2="0.0642871"
+                                  p1="-0.00086158"
+                                  p2="-0.000443529"
+                                  k3="-0.00599387"
+                                  cx="158.0735"
+                                  cy="108.513"
+                                  cx_prime="158.0735"
+        />
+    </xacro:macro>
 </robot>

File: urdf/imu.urdf.xacro (robot description, xacro)
@@ -26,10 +26,10 @@
             <sensor name="s_${name}" type="imu">
                 <always_on>true</always_on>
-                <update_rate>0.0</update_rate>
+<!--                <update_rate>${update_rate}</update_rate>-->
                 <visualize>true</visualize>
                 <plugin filename="libgazebo_ros_imu_sensor.so" name="imu_plugin">
                     <topicName>${name}</topicName>
                     <bodyName>${name}_link</bodyName>
-                    <updateRateHZ>0.0</updateRateHZ>
+                    <updateRateHZ>${update_rate}</updateRateHZ>
                     <gaussianNoise>0.0</gaussianNoise>
                     <xyzOffset>0 0 0</xyzOffset>
